File: pcb/sensor/pspice.sch (KiCad schematic (older format))
At the start: 12 parts, among them U1 OPAMP

Commit message: Sensor spice simulation kicad simulation does not work with opamp multiple ltspice simulations pw_original (RobotShop version) pw_my (My version) pw_ti (My version with sally key bandpass) <= Use this pw_ti2 (Experiments with pw_ti)
Parts:
- removed C1, C2: 1u, symbol Device:C
- removed L2: L_Coupled, symbol Device:L_Coupled
- removed R1, R2, R4: 10k, symbol Device:R
- removed R5: 1M, symbol Device:R
- removed R?: 100M, symbol Device:R
- removed U1: OPAMP, symbol pspice:OPAMP
- added C1: 1u, symbol pspice:CAP
- added C2: 47p, symbol pspice:CAP
- added L1: 85m, symbol pspice:INDUCTOR
- added R1, R2: 10k, symbol pspice:R
- added R4: 300, symbol pspice:R
- R3: value 100k -> 82k; symbol Device:R -> pspice:R
- V1: value VSOURCE -> ac; Spice_Model pulse(0 10 0 0.000001 0.000001 0.00005 0.0001) -> dc 0 ac 100m
Connections:
- net labels added: in, out, v_gnd
- net labels removed: V_GND
- wire segments 37 -> 26
Other:
- note added: "2nd order RLC low pas\nRL Low Pass.\n85mH, 1M => 1.87MHz\n100mH, 100kR => 160kHz"
- note added: "Cant get opamps to work. Use ltspice models"
- note removed: "RL Low Pass.\n85mH, 1M => 1.87MHz\n100mH, 100kR => 160kHz"
- moved on the sheet: R3
