File: pcb/generator/generator.sch (KiCad schematic (older format))
At the start: 28 parts

Commit message: Fix lib in generator schematic
Parts:
- U?: symbol generator-rescue:L6206-local -> local:L6206
Changed lines of the file:
@@
 $EndDescr
 $Comp
-L generator-rescue:L6206-local U?
+L local:L6206 U?
 U 1 1 5CE0D3EB
 P 8400 3050

Commit message: Add generator pcb
Parts:
- removed C?: 100n, symbol Device:C
- removed J?: AVR-ISP-6, symbol Connector:AVR-ISP-6
- removed U?: ATmega328P-AU, Package_QFP:TQFP-32_7x7mm_P0.8mm, symbol MCU_Microchip_ATmega:ATmega328P-AU
- removed U?: R-78HB5.0-0.5, Converter_DCDC:Converter_DCDC_RECOM_R-78HB-0.5_THT, symbol Regulator_Switching:R-78HB5.0-0.5
- added C10, C12, C13: 220n / 100V, Capacitor_THT:C_Disc_D5.1mm_W3.2mm_P5.00mm, symbol Device:C
- added C17: 10n, Capacitor_THT:C_Disc_D4.7mm_W2.5mm_P5.00mm, symbol Device:C
- added C2: 100u / 100V, Capacitor_THT:CP_Radial_D10.0mm_P5.00mm, symbol Device:CP
- added C4, C7: 100n, Capacitor_THT:C_Disc_D4.7mm_W2.5mm_P5.00mm, symbol Device:C
- added D3: Red1, LED_THT:LED_D5.0mm, symbol Device:LED
- added D4: Red2, LED_THT:LED_D5.0mm, symbol Device:LED
- added D5: 5V, Diode_THT:D_DO-15_P10.16mm_Horizontal, symbol Device:D_Zener
- added D6, D7: BAT54, Package_TO_SOT_SMD:SOT-23, symbol Device:D_Schottky_AAK
- added FB1: BLM31KN471SN1L, Inductor_SMD:L_1206_3216Metric, symbol Device:Ferrite_Bead_Small
- added FB2: BLM31SN500SN1, Inductor_SMD:L_1206_3216Metric, symbol Device:Ferrite_Bead_Small
- added FID1, FID2: Fiducial, Fiducial:Fiducial_1.5mm_Mask3mm, symbol Mechanical:Fiducial
- added H1, H2, H3: MountingHole_Pad, MountingHole:MountingHole_3.2mm_M3_Pad, symbol Mechanical:MountingHole_Pad
- added J2: SWD, Connector_PinHeader_1.27mm:PinHeader_2x05_P1.27mm_Vertical, symbol Connector_Generic:Conn_02x05_Odd_Even
- added J5: USB, Connector_USB:USB_Micro-B_Amphenol_10103594-0001LF_Horizontal, symbol Connector:USB_B_Micro
- added R10: 1M, Resistor_THT:R_Axial_DIN0207_L6.3mm_D2.5mm_P7.62mm_Horizontal, symbol Device:R
- added R8, R9: 750R, Resistor_THT:R_Axial_DIN0207_L6.3mm_D2.5mm_P7.62mm_Horizontal, symbol Device:R
- added U1: ATSAMD11D14A-SS, Package_SO:SOIC-20W_7.5x12.8mm_P1.27mm, symbol MCU_Microchip_SAMD:ATSAMD11D14A-SS
- added U2: SRH05S3V3, Converter_DCDC:Converter_DCDC_RECOM_R-78HB-0.5_THT, symbol Regulator_Switching:R-78HB3.3-0.5
- added U4: MCP9700T-HLT, Package_TO_SOT_SMD:SOT-353_SC-70-5, symbol Sensor_Temperature:MCP9700T-HLT
- added U5: LP2985-3.3, Package_TO_SOT_SMD:SOT-23-5, symbol Regulator_Linear:LP2985-3.3
- added U6: SN65220, Package_TO_SOT_SMD:SOT-23-6, symbol Power_Protection:SN65220
- C1: renamed from C?; footprint (none) -> Capacitor_THT:CP_Radial_D10.0mm_P5.00mm; Partnumber (none) -> UVR1J101MPD
- C11: renamed from C?; value 200n / 100V -> 220n / 100V; footprint (none) -> Capacitor_THT:C_Disc_D5.1mm_W3.2mm_P5.00mm; Partnumber (none) -> C322C104M1U5TA
- C14, C15: renamed from C?; value 22p -> 20p; footprint (none) -> Capacitor_THT:C_Disc_D3.8mm_W2.6mm_P2.50mm; Partnumber (none) -> SR151A200JAR
- C16: renamed from C?; footprint (none) -> Capacitor_THT:C_Disc_D4.7mm_W2.5mm_P5.00mm; Partnumber (none) -> K103K10X7RF5UH5
- C18: renamed from C?; footprint (none) -> Capacitor_THT:CP_Radial_D5.0mm_P2.00mm; Partnumber (none) -> TAJC476K020R
- C3, C5, C6: renamed from C?; footprint (none) -> Capacitor_THT:C_Disc_D4.7mm_W2.5mm_P5.00mm; Partnumber (none) -> K104K10X7RF5UH5
- C8: renamed from C?; footprint (none) -> Capacitor_THT:C_Disc_D5.1mm_W3.2mm_P5.00mm; Partnumber (none) -> C322C104M1U5TA
- D1, D2: renamed from D?; footprint (none) -> Diode_THT:D_DO-35_SOD27_P7.62mm_Horizontal; Partnumber (none) -> 1N4148
- J1: renamed from J?; value Conn_01x02 -> Power; footprint (none) -> Connector_Phoenix_MSTB:PhoenixContact_MSTBA_2,5_2-G_1x02_P5.00mm_Horizontal
- J3: renamed from J?; value Conn_01x03 -> CH1; footprint (none) -> Connector_Phoenix_MSTB:PhoenixContact_MSTBA_2,5_3-G-5,08_1x03_P5.08mm_Horizontal
- J4: renamed from J?; value Conn_01x03 -> CH2; footprint (none) -> Connector_Phoenix_MSTB:PhoenixContact_MSTBA_2,5_3-G-5,08_1x03_P5.08mm_Horizontal
- R1, R2, R3, R4, R5: renamed from R?; footprint (none) -> Resistor_THT:R_Axial_DIN0207_L6.3mm_D2.5mm_P7.62mm_Horizontal
- R6, R7: renamed from R?; value R -> 240; footprint (none) -> Resistor_THT:R_Axial_Power_L48.0mm_W12.5mm_P60.96mm; Partnumber (none) -> SQP10AJB-240R
- U3: renamed from U?; value L6206 -> L6206D; footprint (none) -> footprints:PowerSO-36; symbol local:L6206 -> local:L6206P
- Y1: renamed from Y?; value 8MHz -> 32.768kHz; footprint (none) -> Crystal:Crystal_SMD_SeikoEpson_MC146-4Pin_6.7x1.5mm_HandSoldering; symbol Device:Crystal -> Device:Crystal_GND23; Partnumber (none) -> MC-146 32.7680KA-A5: PURE SN
Connections:
- net +48V: now also U3.33 (VS_B), U3.4 (VS_A), C10.2, C12.2, C13.2, C2.1, D7.3 (K), FB2.1, U2.1 (IN); no longer J1.1 (Pin_1), U3.17 (VS_B), U3.20 (VS_A)
- net EN_A: now also U1.6 (PA14)
- net EN_B: now also U1.18 (PA02)
- net ERROR_A: now also U3.13 (OCD_A), U3.8 (EN_A), U1.7 (PA15); no longer U3.23 (EN_A), U3.4 (OCD_A)
- net ERROR_B: now also U3.24 (OCD_B), U3.29 (EN_B), U1.19 (PA03); no longer U3.14 (EN_B), U3.9 (OCD_B)
- net GND: now also C3.1, U3.1 (GND), U3.12 (SENSE_A), U3.25 (SENSE_B), U3.36 (GND), U3.37 (SLUG), Y1.2, Y1.3, C10.1, C12.1, C13.1, C17.1, C2.2, C4.2, C7.2, D5.2 (A), H1.1, H2.1, H3.1, J2.3 (Pin_3), J2.5 (Pin_5), J2.9 (Pin_9), J5.5 (GND), R10.2, U1.16 (GND), U2.2 (GND), U4.2 (GND), U5.2 (GND), U6.2 (GND), U6.5 (GND); no longer C3.2, U3.10 (SENSE_B), U3.3 (SENSE_A), U3.6 (GND), U3.7 (GND)
- net IN1_A: now also U3.10 (IN1_A), U1.2 (PA06); no longer U3.1 (IN1_A)
- net IN1_B: now also U3.26 (IN1_B), U1.20 (PA04); no longer U3.11 (IN1_B)
- net IN2_A: now also U3.11 (IN2_A), U1.3 (PA07); no longer U3.2 (IN2_A)
- net IN2_B: now also U3.27 (IN2_B), U1.1 (PA05); no longer U3.12 (IN2_B)
- net at R5.2: now also U3.28 (PROGCL_B); no longer U3.13 (PROGCL_B)
- net at C8.1, D2.1 (K): now also U3.30 (VBOOT); no longer U3.15 (VBOOT)
- net at J4.1 (Pin_1): now also U3.32 (OUT2_B); no longer U3.16 (OUT2_B)
- net at J3.1 (Pin_1): now also U3.5 (OUT2_A); no longer U3.21 (OUT2_A)
- net at U3.22 (OUT1_B): now also J4.2 (Pin_2), R7.2; no longer C16.1
- net at R4.1: now also U3.9 (PROGCL_A); no longer U3.24 (PROGCL_A)
- net at J3.2 (Pin_2), R6.2: now also U3.15 (OUT1_A); no longer U3.5 (OUT1_A)
- net at C15.2: now also Y1.4, U1.5 (PA09/XOUT); no longer Y1.1
- net at C14.1: now also Y1.1, U1.4 (PA08/XIN); no longer Y1.2
- net +5V renamed +3V3
- net +3V3: now also C3.2, C7.1, D3.2 (A), D4.2 (A), D6.1 (A), D6.2 (A), D7.1 (A), D7.2 (A), J2.1 (Pin_1), U1.17 (VDD), U2.3 (OUT), U4.4 (Vdd), U5.5 (VOUT); no longer C3.1
- new net: C16.1, U3.7 (VCP)
- new net: FB2.2, J1.1 (Pin_1)
- new net: D4.1 (K), R9.1
- new net: D3.1 (K), R8.1
- new net: R8.2, U1.9 (PA22)
- new net: R9.2, U1.10 (PA23)
- new net: C4.1, D6.3 (K), FB1.1, U5.1 (VIN), U5.3 (ON/~OFF~)
- new net: D5.1 (K), FB1.2, J5.1 (VBUS)
- new net: C17.2, J5.6 (Shield), R10.1
- new net R_TEMP: U1.8 (PA16), U4.3 (Vout)
- new net SWCLK: J2.4 (Pin_4), U1.12 (PA30/SWCLK)
- new net SWDIO: J2.2 (Pin_2), U1.13 (PA31/SWDIO)
- new net USB_D+: J5.3 (D+), U1.15 (PA25), U6.1, U6.6 (A)
- new net USB_D-: J5.2 (D-), U1.14 (PA24), U6.3, U6.4 (B)
- new net ~RESET: J2.10 (Pin_10), U1.11 (PA28/~RST)
- no-connect marks 13 -> 5
Other:
- note added: "N/C pins used for better routing\n(see datasheet)"
- note added: "Overcurrent Limit of approx. 1A\nNo current sense resistor"
- note added: "Pin3:\nResistor limits current for short wires.\n10W @ 2x24V = 0,2A => 240Ohm\nThis resistor won't survive 2x48V short circuit!"
- note added: "USB and 48V power source are connected to create a ORed power\nschema. This enables to program the system without 48V present.\nThe diodes prevent reverse output faults."
- note removed: "Use ATTINY48-AUR ?\nAdd LEDs for status\nAdd configuration"
- moved on the sheet: C1, C14, C15, C18, C3, J1

Commit message: Release preparation
Parts:
- FB1: value BLM31KN471SN1L -> BLM31KN471SN1L
Changed lines of the file:
@@
 encoding utf-8
 Sheet 1 1
-Title ""
-Date ""
-Rev ""
-Comp ""
+Title "Perimeter Wire Generator"
+Date "2019-09-02"
+Rev "R1"
+Comp "Meadow Robotics GmbH"
 Comment1 ""
 Comment2 ""
@@
 P 2450 2550
 F 0 "FB1" V 2213 2550 50  0000 C CNN
-F 1 " BLM31KN471SN1L" V 2304 2550 50  0000 C CNN
+F 1 "BLM31KN471SN1L" V 2304 2550 50  0000 C CNN
 F 2 "Inductor_SMD:L_1206_3216Metric" V 2380 2550 50  0001 C CNN
 F 3 "~" H 2450 2550 50  0001 C CNN
