File: pcb/generator/generator.sch (KiCad schematic (older format))
At the start: 75 parts, among them J1 Power, J2 SWD, J3 CH1, J4 CH2, J5 USB, J6 Au, J7 Bu, J8 Al, J9 Bl, U1 ATSAMD21E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

Commit message: gernerator pcb r2 - place references - adjust mask clearance
Parts:
- U1: Partnumber (none) -> ATSAMD21E17D
Changed lines of the file:
@@
 Sheet 1 1
 Title "Perimeter Wire Generator"
-Date "2019-09-02"
-Rev "R1"
+Date "2020-01-18"
+Rev "R2"
 Comp "Meadow Robotics GmbH"
 Comment1 ""
@@
 F 2 "Package_QFP:TQFP-32_7x7mm_P0.8mm" H 2650 5600 50  0001 C CNN
 F 3 "http://ww1.microchip.com/downloads/en/DeviceDoc/SAMD21-Family-DataSheet-DS40001882D.pdf" H 3350 7350 50  0001 C CNN
+F 4 "ATSAMD21E17D" H 3350 6350 50  0001 C CNN "Partnumber"
 	1    3350 6350
 	1    0    0    -1
