File: pcb/generator/generator.sch (KiCad schematic (older format))
At the start: 75 parts, among them J1 Power, J2 SWD, J3 CH1, J4 CH2, J5 USB, J6 Au, J7 Bu, J8 Al, J9 Bl, U1 ATSAMD21E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

Commit message: generator: Update parnumbers (for r2)
Parts:
- C18: Partnumber TAJC476K020R -> TAJC476K020RNJ
- D3, D4: Partnumber CLMVC-FKA -> CLMVC-FKA-CL1D1L71BB7C3C3
- FB2: Partnumber BLM31SN500SN1 -> BLM31SN500SN1L
- U1: Partnumber ATSAMD21E17D -> ATSAMD21E17D-AU
Changed lines of the file:
@@
 F 2 "Capacitor_Tantalum_SMD:CP_EIA-6032-28_Kemet-C" H 2588 1400 50  0001 C CNN
 F 3 "~" H 2550 1550 50  0001 C CNN
-F 4 "TAJC476K020R" H 2550 1550 50  0001 C CNN "Partnumber"
+F 4 "TAJC476K020RNJ" H 2550 1550 50  0001 C CNN "Partnumber"
 	1    2550 1550
 	1    0    0    -1
@@
 F 2 "Inductor_SMD:L_1206_3216Metric" V 8880 800 50  0001 C CNN
 F 3 "~" H 8950 800 50  0001 C CNN
-F 4 "BLM31SN500SN1" H 8950 800 50  0001 C CNN "Partnumber"
+F 4 "BLM31SN500SN1L" H 8950 800 50  0001 C CNN "Partnumber"
 	1    8950 800
 	0    1    1    0
@@
 F 2 "Package_QFP:TQFP-32_7x7mm_P0.8mm" H 2650 5600 50  0001 C CNN
 F 3 "http://ww1.microchip.com/downloads/en/DeviceDoc/SAMD21-Family-DataSheet-DS40001882D.pdf" H 3350 7350 50  0001 C CNN
-F 4 "ATSAMD21E17D" H 3350 6350 50  0001 C CNN "Partnumber"
+F 4 "ATSAMD21E17D-AU" H 3350 6350 50  0001 C CNN "Partnumber"
 	1    3350 6350
 	1    0    0    -1
@@
 F 2 "LED_SMD:LED_Cree-PLCC4_2x2mm_CW" H 4950 4780 50  0001 L CNN
 F 3 "" H 4950 4700 50  0001 L CNN
-F 4 "CLMVC-FKA" H 5150 5100 50  0001 C CNN "Partnumber"
+F 4 "CLMVC-FKA-CL1D1L71BB7C3C3" H 5150 5100 50  0001 C CNN "Partnumber"
 	1    5150 5100
 	1    0    0    1
@@
 F 2 "LED_SMD:LED_Cree-PLCC4_2x2mm_CW" H 5300 5630 50  0001 L CNN
 F 3 "" H 5300 5550 50  0001 L CNN
-F 4 "CLMVC-FKA" H 5500 5950 50  0001 C CNN "Partnumber"
+F 4 "CLMVC-FKA-CL1D1L71BB7C3C3" H 5500 5950 50  0001 C CNN "Partnumber"
 	1    5500 5950
 	1    0    0    1

Commit message: generator pcb: replace SMBJ48CA with SMBJ48A
Parts:
- D8: Partnumber SMBJ48CATR -> SMBJ48ATR
Changed lines of the file:
@@
 F 2 "Diode_SMD:D_SMB" H 8700 950 50  0001 C CNN
 F 3 "~" H 8700 950 50  0001 C CNN
-F 4 "SMBJ48CATR" V 8700 950 50  0001 C CNN "Partnumber"
+F 4 "SMBJ48ATR" V 8700 950 50  0001 C CNN "Partnumber"
 	1    8700 950
 	0    1    1    0
